Commit message: Fixed simulation of the arm

File: tb_description/urdf/smart_arm.xacro (robot description, xacro)
@@ -266,5 +266,5 @@
           <type>transmission_interface/SimpleTransmission</type>
           <joint name="shoulder_pan_joint"/>
-            <actuator name="shoulder_pan_motor">
+          <actuator name="shoulder_pan_motor">
             <hardwareInterface>PositionJointInterface</hardwareInterface>
             <mechanicalReduction>1.0</mechanicalReduction>
@@ -273,5 +273,5 @@
         <transmission name="shoulder_pitch_trans">
           <type>transmission_interface/SimpleTransmission</type>
-          <joint name="shoulder_pan_joint"/>
+          <joint name="shoulder_pitch_joint"/>
             <actuator name="shoulder_pitch_motor">
             <hardwareInterface>PositionJointInterface</hardwareInterface>
