Commit message: Update.

File: tb_description/robots/turtlebot.urdf.xacro (robot description, xacro)
@@ -5,5 +5,4 @@
        xmlns:interface="http://playerstage.sourceforge.net/gazebo/xmlschema/#interface"
        xmlns:xacro="http://ros.org/wiki/xacro">
-  <include filename="$(find tb_description)/urdf/turtlebot_hardware.urdf.xacro" />
   <include filename="$(find tb_description)/urdf/turtlebot_body.urdf.xacro" />
   <include filename="$(find tb_description)/urdf/turtlebot_calibration.xacro" />

File: tb_description/urdf/turtlebot_body.urdf.xacro (robot description, xacro)
@@ -3,5 +3,5 @@
   <property name="M_PI" value="3.14159"/>
   <!-- Macro for TurtleBot body. Including Gazebo extensions, but does not include Kinect -->
-  <include filename="$(find btb_description)/urdf/gazebo.urdf.xacro"/>
+  <include filename="$(find tb_description)/urdf/gazebo.urdf.xacro"/>
   <property name="base_x" value="0.33" />
   <property name="base_y" value="0.33" />

File: tb_description/urdf/turtlebot_kinect.urdf.xacro (robot description, xacro)
@@ -27,5 +27,5 @@
       <origin xyz=" 0 0 0 " rpy="0 0 0" />
       <geometry>
-        <mesh filename="package://btb_description/meshes/kinect.dae"/>
+        <mesh filename="package://tb_description/meshes/kinect.dae"/>
       </geometry>
     </visual>

Commit message: updates for new Gazebo

File: tb_description/robots/turtlebot.urdf.xacro (robot description, xacro)
@@ -5,11 +5,11 @@
        xmlns:interface="http://playerstage.sourceforge.net/gazebo/xmlschema/#interface"
        xmlns:xacro="http://ros.org/wiki/xacro">
-  <include filename="$(find tb_description)/urdf/turtlebot_body.urdf.xacro" />
-  <include filename="$(find tb_description)/urdf/turtlebot_calibration.xacro" />
-  <include filename="$(find tb_description)/urdf/turtlebot_kinect.urdf.xacro" />
-  <include filename="$(find tb_description)/urdf/smart_arm.xacro" />
-  <include filename="$(find tb_description)/urdf/constants.xacro" />
+  <xacro:include filename="$(find tb_description)/urdf/turtlebot_body.urdf.xacro" />
+  <xacro:include filename="$(find tb_description)/urdf/turtlebot_calibration.xacro" />
+  <xacro:include filename="$(find tb_description)/urdf/turtlebot_kinect.urdf.xacro" />
+  <xacro:include filename="$(find tb_description)/urdf/smart_arm.xacro" />
+  <xacro:include filename="$(find tb_description)/urdf/constants.xacro" />
   <gazebo>
-     <controller:gazebo_ros_controller_manager name="gazebo_ros_controller_manager" plugin="libgazebo_ros_controller_manager.so">
+     <!--controller:gazebo_ros_controller_manager name="gazebo_ros_controller_manager" plugin="libgazebo_ros_controller_manager.so">
           <alwaysOn>true</alwaysOn>
           <updateRate>1000.0</updateRate>
@@ -17,30 +17,8 @@
           <robotParam>robot_description</robotParam>
           <interface:audio name="gazebo_ros_controller_manager_dummy_iface" />
-     </controller:gazebo_ros_controller_manager>
-     <!--controller:gazebo_ros_p3d name="p3d_base_controller" plugin="libgazebo_ros_p3d.so">
-         <alwaysOn>true</alwaysOn>
-         <updateRate>100.0</updateRate>
-         <bodyName>base_link</bodyName>
-         <topicName>base_pose_ground_truth</topicName>
-         <gaussianNoise>0.0</gaussianNoise>
-         <frameName>map</frameName>
-         <xyzOffsets>0 0 0</xyzOffsets>
-         <rpyOffsets>0 0 0</rpyOffsets>
-         <interface:position name="p3d_base_position"/>
-     </controller:gazebo_ros_p3d-->
-     <!-- just for inspiration -->
-     <!--controller:gazebo_ros_power_monitor name="gazebo_ros_power_monitor_controller" plugin="libgazebo_ros_power_monitor.so">
-      <alwaysOn>true</alwaysOn>
-      <updateRate>1.0</updateRate>
-      <timeout>5</timeout>
-      <interface:audio name="power_monitor_dummy_interface" />
-      <powerStateTopic>power_state</powerStateTopic>
-      <powerStateRate>10.0</powerStateRate>
-      <fullChargeCapacity>87.78</fullChargeCapacity>
-      <dischargeRate>-474</dischargeRate>
-      <chargeRate>525</chargeRate>
-      <dischargeVoltage>15.52</dischargeVoltage>
-      <chargeVoltage>16.41</chargeVoltage>
-    </controller:gazebo_ros_power_monitor-->
+     </controller:gazebo_ros_controller_manager-->
+    <plugin name="gazebo_ros_control" filename="libgazebo_ros_control.so">
+      <robotNamespace>dynamixel</robotNamespace>
+    </plugin>
   </gazebo>
   <!-- Body of TurtleBot, with plates, standoffs and Create (including sim sensors) -->

File: tb_description/urdf/gazebo.urdf.xacro (robot description, xacro)
@@ -2,5 +2,5 @@
 <robot xmlns:controller="http://playerstage.sourceforge.net/gazebo/xmlschema/#controller" xmlns:interface="http://playerstage.sourceforge.net/gazebo/xmlschema/#interface" xmlns:sensor="http://playerstage.sourceforge.net/gazebo/xmlschema/#sensor" xmlns:xacro="http://ros.org/wiki/xacro" name="turtlebot_gazebo">
 <xacro:macro name="turtlebot_sim_kinect">
-  <gazebo reference="camera_link">
+  <!--gazebo reference="camera_link">
     <sensor:camera name="camera">
       <imageFormat>R8G8B8</imageFormat>
@@ -28,5 +28,28 @@
       </controller:gazebo_ros_openni_kinect>
     </sensor:camera>
-  </gazebo>
+  </gazebo-->
+  <plugin name="kinect_controller" filename="libgazebo_ros_openni_kinect.so">
+    <baseline>0.2</baseline>
+    <alwaysOn>true</alwaysOn>
+    <updateRate>1.0</updateRate>
+    <cameraName>camera_ir</cameraName>
+    <imageTopicName>/cam3d/depth/image_raw</imageTopicName>
+    <cameraInfoTopicName>/cam3d/depth/camera_info</cameraInfoTopicName>
+    <depthImageTopicName>/cam3d/depth/image_raw</depthImageTopicName>
+    <depthImageInfoTopicName>/cam3d/depth/camera_info</depthImageInfoTopicName>
+    <pointCloudTopicName>/cam3d/depth/points</pointCloudTopicName>
+    <frameName>camera_link</frameName>
+    <pointCloudCutoff>0.5</pointCloudCutoff>
+    <distortionK1>0.00000001</distortionK1>
+    <distortionK2>0.00000001</distortionK2>
+    <distortionK3>0.00000001</distortionK3>
+    <distortionT1>0.00000001</distortionT1>
+    <distortionT2>0.00000001</distortionT2>
+    <CxPrime>0</CxPrime>
+    <Cx>0</Cx>
+    <Cy>0</Cy>
+    <focalLength>0</focalLength>
+    <hackBaseline>0</hackBaseline>
+  </plugin>
   <transmission type="pr2_mechanism_model/SimpleTransmission" name="kinect_trans">
     <actuator name="kinect_motor" />
@@ -42,9 +65,9 @@
 </xacro:macro>
 <xacro:macro name="turtlebot_sim_imu_left">
-  <gazebo>
+  <!--gazebo>
     <controller:gazebo_ros_imu name="imu_controller" plugin="libgazebo_ros_imu.so">
       <alwaysOn>true</alwaysOn>
       <updateRate>30</updateRate>
-      <bodyName>imu_left_link</bodyName> <!-- was gyro_link -->
+      <bodyName>imu_left_link</bodyName>
       <topicName>imu_left/data</topicName>
       <gaussianNoise>${0.0017*0.0017}</gaussianNoise>
@@ -53,12 +76,12 @@
       <interface:position name="imu_left_position"/>
     </controller:gazebo_ros_imu>
-  </gazebo>
+  </gazebo-->
 </xacro:macro>
 <xacro:macro name="turtlebot_sim_imu_right">
-  <gazebo>
+  <!--gazebo>
     <controller:gazebo_ros_imu name="imu_controller" plugin="libgazebo_ros_imu.so">
       <alwaysOn>true</alwaysOn>
       <updateRate>30</updateRate>
-      <bodyName>imu_right_link</bodyName> <!-- was gyro_link -->
+      <bodyName>imu_right_link</bodyName>
       <topicName>imu_right/data</topicName>
       <gaussianNoise>${0.0017*0.0017}</gaussianNoise>
@@ -67,10 +90,10 @@
       <interface:position name="imu_right_position"/>
     </controller:gazebo_ros_imu>
-  </gazebo>
+  </gazebo-->
 </xacro:macro>
 <xacro:macro name="turtlebot_sim_laser">
-  <gazebo reference="laser">
+  <!--gazebo reference="laser">
     <sensor:ray name="laser">
-      <rayCount>540</rayCount> <!-- 270 deg. / 0.5 deg. -->
+      <rayCount>540</rayCount>
       <rangeCount>540</rangeCount>
       <laserCount>1</laserCount>
@@ -92,9 +115,44 @@
       </controller:gazebo_ros_laser>
     </sensor:ray>
+  </gazebo-->
+  <gazebo reference="laser">
+    <sensor type="gpu_ray" name="sick_sensor">
+      <pose>0 0 0 0 0 0</pose>
+      <visualize>false</visualize>
+      <update_rate>20</update_rate>
+      <ray>
+        <scan>
+          <horizontal>
+            <samples>540</samples>
+            <resolution>1</resolution>
+            <min_angle>-1.570796</min_angle>
+            <max_angle>1.570796</max_angle>
+          </horizontal>
+        </scan>
+        <range>
+          <min>0.10</min>
+          <max>30.0</max>
+          <resolution>0.01</resolution>
+        </range>
+        <noise>
+          <type>gaussian</type>
+          <!-- Noise parameters based on published spec for Hokuyo laser
+               achieving "+-30mm" accuracy at range < 10m.  A mean of 0.0m and
+               stddev of 0.01m will put 99.7% of samples within 0.03m of the true
+               reading. -->
+          <mean>0.0</mean>
+          <stddev>0.01</stddev>
+        </noise>
+      </ray>
+      <plugin name="gazebo_ros_head_hokuyo_controller" filename="libgazebo_ros_gpu_laser.so">
+        <topicName>scan</topicName>
+        <frameName>laser</frameName>
+      </plugin>
+    </sensor>
   </gazebo>
 </xacro:macro>
 <xacro:macro name="turtlebot_sim_create">
   <gazebo>
-    <controller:gazebo_ros_create name="create_controller" plugin="libgazebo_ros_create.so">
+    <!--controller:gazebo_ros_create name="create_controller" plugin="libgazebo_ros_create.so">
       <alwaysOn>true</alwaysOn>
       <node_namespace>turtlebot_node</node_namespace>
@@ -108,22 +166,22 @@
       <updateRate>40</updateRate>
       <torque>1.0</torque>
-    </controller:gazebo_ros_create>
-    <!--controller:diffdrive_plugin name="differential_drive_controller" plugin="libdiffdrive_plugin.so">
-       <alwaysOn>true</alwaysOn>
-       <update>100</update>
-       <updateRate>100.0</updateRate>
-       <leftJoint>left_wheel_joint</leftJoint>
-       <rightJoint>right_wheel_joint</rightJoint>
-       <wheelSeparation>.260</wheelSeparation>
-       <wheelDiameter>0.066</wheelDiameter>
-       <torque>1.0</torque>
-       <interface:position name="position_iface_0"/>
-       <robotNamespace></robotNamespace>
-       <topicName>cmd_vel</topicName>
-    </controller:diffdrive_plugin-->
+    </controller:gazebo_ros_create-->
+    <plugin name="differential_drive_controller" filename="libgazebo_ros_diff_drive.so">
+    <alwaysOn>true</alwaysOn>
+    <updateRate>40</updateRate>
+    <leftJoint>left_wheel_joint</leftJoint>
+    <rightJoint>right_wheel_joint</rightJoint>
+    <wheelSeparation>.260</wheelSeparation>
+    <wheelDiameter>0.066</wheelDiameter>
+    <torque>1.0</torque>
+    <commandTopic>cmd_vel</commandTopic>
+    <odometryTopic>odom</odometryTopic>
+    <odometryFrame>odom</odometryFrame>
+    <robotBaseFrame>base_footprint</robotBaseFrame>
+  </plugin>
   </gazebo>
 </xacro:macro>
 <xacro:macro name="turtlebot_sim_wall_sensors">
-  <gazebo reference="wall_sensor_link">
+  <!--gazebo reference="wall_sensor_link">
     <sensor:ray name="wall_sensor">
       <alwaysActive>true</alwaysActive>
@@ -189,5 +247,5 @@
       <displayRays>fan</displayRays>
     </sensor:ray>
-  </gazebo>
+  </gazebo-->
   </xacro:macro>
   <gazebo reference="left_wheel_link">
@@ -196,5 +254,5 @@
     <kp value="100000000.0"/>
     <kd value="10000.0"/>
-    <fdir value="1 0 0"/>
+    <!--fdir value="1 0 0"/-->
   </gazebo>
   <gazebo reference="right_wheel_link">
@@ -203,5 +261,5 @@
     <kp value="100000000.0"/>
     <kd value="10000.0"/>
-    <fdir value="1 0 0"/>
+    <!--fdir value="1 0 0"/-->
   </gazebo>
   <gazebo reference="rear_wheel_link">

File: tb_description/urdf/smart_arm.xacro (robot description, xacro)
@@ -33,10 +33,7 @@
 * Author: Antons Rebguns
 -->
-<robot
-    xmlns:sensor="http://playerstage.sourceforge.net/gazebo/xmlschema/#sensor"
-    xmlns:controller="http://playerstage.sourceforge.net/gazebo/xmlschema/#controller"
-    xmlns:interface="http://playerstage.sourceforge.net/gazebo/xmlschema/#interface">
-    <include filename="$(find smart_arm_description)/urdf/materials.urdf.xacro" />
-    <macro name="smart_arm" params="parent *origin">
+<robot name="smart_arm_robot" xmlns:xacro="http://www.ros.org/wiki/xacro">
+    <xacro:include filename="$(find smart_arm_description)/urdf/materials.urdf.xacro" />
+    <xacro:macro name="smart_arm" params="parent *origin">
         <!-- ****** JOINT DEFINITIONS ****** -->
         <!-- Arm's base joint -->
@@ -382,4 +379,4 @@
             <fudgeFactor value="1.0" />
         </gazebo>
-    </macro>
+    </xacro:macro>
 </robot>

File: tb_description/urdf/turtlebot_body.urdf.xacro (robot description, xacro)
@@ -3,5 +3,5 @@
   <property name="M_PI" value="3.14159"/>
   <!-- Macro for TurtleBot body. Including Gazebo extensions, but does not include Kinect -->
-  <include filename="$(find tb_description)/urdf/gazebo.urdf.xacro"/>
+  <xacro:include filename="$(find tb_description)/urdf/gazebo.urdf.xacro"/>
   <property name="base_x" value="0.33" />
   <property name="base_y" value="0.33" />
@@ -301,5 +301,4 @@
       <geometry>
         <box size="0.1 0.1 0.15" />
-        <!--mesh filename="package://btb_description/meshes/sick_s300_laser.dae"/-->
       </geometry>
       <material name="blue">

File: tb_description/urdf/turtlebot_kinect.urdf.xacro (robot description, xacro)
@@ -1,6 +1,6 @@
 <?xml version="1.0"?>
 <robot name="turtlebot_hardware" xmlns:xacro="http://ros.org/wiki/xacro">
-  <include filename="$(find tb_description)/urdf/gazebo.urdf.xacro"/>
-  <include filename="$(find tb_description)/urdf/turtlebot_calibration.xacro" />
+  <xacro:include filename="$(find tb_description)/urdf/gazebo.urdf.xacro"/>
+  <xacro:include filename="$(find tb_description)/urdf/turtlebot_calibration.xacro" />
 <xacro:macro name="turtlebot_kinect">
   <joint name="kinect_joint" type="revolute">

Commit message: Fixes for Gazebo 1.9

File: tb_description/robots/turtlebot.urdf.xacro (robot description, xacro)
@@ -19,5 +19,5 @@
      </controller:gazebo_ros_controller_manager-->
     <plugin name="gazebo_ros_control" filename="libgazebo_ros_control.so">
-      <robotNamespace>dynamixel</robotNamespace>
+      <robotNamespace>/dynamixel</robotNamespace>
     </plugin>
   </gazebo>
@@ -29,3 +29,4 @@
   <!-- Kinect frames and mounting (includes simulation) -->
   <turtlebot_kinect/>
+  <turtlebot_sim_kinect/>
 </robot>

File: tb_description/urdf/gazebo.urdf.xacro (robot description, xacro)
@@ -52,9 +52,17 @@
     <hackBaseline>0</hackBaseline>
   </plugin>
-  <transmission type="pr2_mechanism_model/SimpleTransmission" name="kinect_trans">
+  <!--transmission type="pr2_mechanism_model/SimpleTransmission" name="kinect_trans">
     <actuator name="kinect_motor" />
     <joint name="kinect_joint" />
     <mechanicalReduction>1.0</mechanicalReduction>
     <motorTorqueConstant>1.0</motorTorqueConstant>
+  </transmission-->
+  <transmission name="kinect_trans">
+    <type>transmission_interface/SimpleTransmission</type>
+    <joint name="kinect_joint"/>
+      <actuator name="kinect_motor">
+      <hardwareInterface>PositionJointInterface</hardwareInterface>
+      <mechanicalReduction>1.0</mechanicalReduction>
+    </actuator>
   </transmission>
   <gazebo reference="kinect_joint">

File: tb_description/urdf/smart_arm.xacro (robot description, xacro)
@@ -263,39 +263,51 @@
         </link>
         <!-- ****** TRANSMISSION DEFINITIONS ****** -->
-        <transmission type="pr2_mechanism_model/SimpleTransmission" name="shoulder_pan_trans">
-            <actuator name="shoulder_pan_motor" />
-            <joint name="shoulder_pan_joint" />
-            <mechanicalReduction>1.0</mechanicalReduction>
-            <motorTorqueConstant>1.0</motorTorqueConstant>
-        </transmission>
-        <transmission type="pr2_mechanism_model/SimpleTransmission" name="shoulder_pitch_trans">
-            <actuator name="shoulder_pitch_motor" />
-            <joint name="shoulder_pitch_joint" />
-            <mechanicalReduction>1.0</mechanicalReduction>
-            <motorTorqueConstant>1.0</motorTorqueConstant>
-        </transmission>
-        <transmission type="pr2_mechanism_model/SimpleTransmission" name="elbow_flex_trans">
-            <actuator name="elbow_flex_motor" />
-            <joint name="elbow_flex_joint" />
-            <mechanicalReduction>1.0</mechanicalReduction>
-            <motorTorqueConstant>1.0</motorTorqueConstant>
-        </transmission>
-        <transmission type="pr2_mechanism_model/SimpleTransmission" name="wrist_roll_trans">
-            <actuator name="wrist_roll_motor" />
-            <joint name="wrist_roll_joint" />
-            <mechanicalReduction>1.0</mechanicalReduction>
-            <motorTorqueConstant>1.0</motorTorqueConstant>
-        </transmission>
-        <transmission type="pr2_mechanism_model/SimpleTransmission" name="right_finger_trans">
-            <actuator name="right_finger_motor" />
-            <joint name="right_finger_joint" />
-            <mechanicalReduction>1.0</mechanicalReduction>
-            <motorTorqueConstant>1.0</motorTorqueConstant>
-        </transmission>
-        <transmission type="pr2_mechanism_model/SimpleTransmission" name="left_finger_trans">
-            <actuator name="left_finger_motor" />
-            <joint name="left_finger_joint" />
-            <mechanicalReduction>1.0</mechanicalReduction>
-            <motorTorqueConstant>1.0</motorTorqueConstant>
+        <transmission name="shoulder_pan_trans">
+          <type>transmission_interface/SimpleTransmission</type>
+          <joint name="shoulder_pan_joint"/>
+            <actuator name="shoulder_pan_motor">
+            <hardwareInterface>PositionJointInterface</hardwareInterface>
+            <mechanicalReduction>1.0</mechanicalReduction>
+          </actuator>
+        </transmission>
+        <transmission name="shoulder_pitch_trans">
+          <type>transmission_interface/SimpleTransmission</type>
+          <joint name="shoulder_pan_joint"/>
+            <actuator name="shoulder_pitch_motor">
+            <hardwareInterface>PositionJointInterface</hardwareInterface>
+            <mechanicalReduction>1.0</mechanicalReduction>
+          </actuator>
+        </transmission>
+        <transmission name="elbow_flex_trans">
+          <type>transmission_interface/SimpleTransmission</type>
+          <joint name="elbow_flex_joint"/>
+            <actuator name="elbow_flex_motor">
+            <hardwareInterface>PositionJointInterface</hardwareInterface>
+            <mechanicalReduction>1.0</mechanicalReduction>
+          </actuator>
+        </transmission>
+        <transmission name="wrist_roll_trans">
+          <type>transmission_interface/SimpleTransmission</type>
+          <joint name="wrist_roll_joint"/>
+            <actuator name="wrist_roll_motor">
+            <hardwareInterface>PositionJointInterface</hardwareInterface>
+            <mechanicalReduction>1.0</mechanicalReduction>
+          </actuator>
+        </transmission>
+        <transmission name="right_finger_trans">
+          <type>transmission_interface/SimpleTransmission</type>
+          <joint name="right_finger_joint"/>
+            <actuator name="right_finger_motor">
+            <hardwareInterface>PositionJointInterface</hardwareInterface>
+            <mechanicalReduction>1.0</mechanicalReduction>
+          </actuator>
+        </transmission>
+        <transmission name="left_finger_trans">
+          <type>transmission_interface/SimpleTransmission</type>
+          <joint name="left_finger_joint"/>
+            <actuator name="left_finger_motor">
+            <hardwareInterface>PositionJointInterface</hardwareInterface>
+            <mechanicalReduction>1.0</mechanicalReduction>
+          </actuator>
         </transmission>
         <!-- ****** MATERIAL DEFINITIONS ****** -->

File: tb_description/urdf/turtlebot_body.urdf.xacro (robot description, xacro)
@@ -43,5 +43,5 @@
       <origin xyz=" 0 0 0.0308" rpy="0 0 0" />
       <geometry>
-        <mesh filename="package://turtlebot_description/meshes/create_body.dae"/>
+        <mesh filename="package://create_description/meshes/create_body.dae"/>
       </geometry>
     </visual>
