Commit message: kinect fixed

File: tb_description/robots/turtlebot.urdf.xacro (robot description, xacro)
@@ -10,4 +10,5 @@
   <xacro:include filename="$(find tb_description)/urdf/smart_arm.xacro" />
   <xacro:include filename="$(find tb_description)/urdf/constants.xacro" />
+  <xacro:include filename="$(find tb_description)/urdf/gazebo.urdf.xacro" />
   <gazebo>
      <!--controller:gazebo_ros_controller_manager name="gazebo_ros_controller_manager" plugin="libgazebo_ros_controller_manager.so">
@@ -24,4 +25,6 @@
   <!-- Body of TurtleBot, with plates, standoffs and Create (including sim sensors) -->
   <turtlebot_body/>
+  <!--turtlebot_sim_imu_left/>
+  <turtlebot_sim_imu_right/-->
    <smart_arm parent="base_link">
      <origin xyz="0.13 0 0.12" rpy="0 0 0" />
@@ -29,4 +32,3 @@
   <!-- Kinect frames and mounting (includes simulation) -->
   <turtlebot_kinect/>
-  <turtlebot_sim_kinect/>
 </robot>

File: tb_description/urdf/gazebo.urdf.xacro (robot description, xacro)
@@ -2,60 +2,46 @@
 <robot xmlns:controller="http://playerstage.sourceforge.net/gazebo/xmlschema/#controller" xmlns:interface="http://playerstage.sourceforge.net/gazebo/xmlschema/#interface" xmlns:sensor="http://playerstage.sourceforge.net/gazebo/xmlschema/#sensor" xmlns:xacro="http://ros.org/wiki/xacro" name="turtlebot_gazebo">
 <xacro:macro name="turtlebot_sim_kinect">
-  <!--gazebo reference="camera_link">
-    <sensor:camera name="camera">
-      <imageFormat>R8G8B8</imageFormat>
-      <imageSize>640 480</imageSize>
-      <hfov>57</hfov>
-      <nearClip>0.4</nearClip>
-      <farClip>100.0</farClip>
-      <updateRate>5</updateRate>
-      <baseline>0.2</baseline>
-      <controller:gazebo_ros_openni_kinect name="kinect_camera_controller" plugin="libgazebo_ros_openni_kinect.so">
-        <alwaysOn>true</alwaysOn>
-        <updateRate>5</updateRate>
-        <pointCloudCutOff>0.4</pointCloudCutOff>
-        <imageTopicName>/cam3d/rgb/image_color</imageTopicName>
-        <pointCloudTopicName>/cam3d/depth/points</pointCloudTopicName>
-        <cameraInfoTopicName>/cam3d/camera_info</cameraInfoTopicName>
-        <depthImageTopicName>/cam3d/depth/image</depthImageTopicName>
-        <depthImageInfoTopicName>/cam3d/depth/camera_info</depthImageInfoTopicName>
-        <frameName>camera_rgb_optical_frame</frameName>
-        <distortion_k1>0.00000001</distortion_k1>
-        <distortion_k2>0.00000001</distortion_k2>
-        <distortion_k3>0.00000001</distortion_k3>
-        <distortion_t1>0.00000001</distortion_t1>
-        <distortion_t2>0.00000001</distortion_t2>
-      </controller:gazebo_ros_openni_kinect>
-    </sensor:camera>
-  </gazebo-->
-  <plugin name="kinect_controller" filename="libgazebo_ros_openni_kinect.so">
-    <baseline>0.2</baseline>
-    <alwaysOn>true</alwaysOn>
-    <updateRate>1.0</updateRate>
-    <cameraName>camera_ir</cameraName>
-    <imageTopicName>/cam3d/depth/image_raw</imageTopicName>
-    <cameraInfoTopicName>/cam3d/depth/camera_info</cameraInfoTopicName>
-    <depthImageTopicName>/cam3d/depth/image_raw</depthImageTopicName>
-    <depthImageInfoTopicName>/cam3d/depth/camera_info</depthImageInfoTopicName>
-    <pointCloudTopicName>/cam3d/depth/points</pointCloudTopicName>
-    <frameName>camera_link</frameName>
-    <pointCloudCutoff>0.5</pointCloudCutoff>
-    <distortionK1>0.00000001</distortionK1>
-    <distortionK2>0.00000001</distortionK2>
-    <distortionK3>0.00000001</distortionK3>
-    <distortionT1>0.00000001</distortionT1>
-    <distortionT2>0.00000001</distortionT2>
-    <CxPrime>0</CxPrime>
-    <Cx>0</Cx>
-    <Cy>0</Cy>
-    <focalLength>0</focalLength>
-    <hackBaseline>0</hackBaseline>
-  </plugin>
-  <!--transmission type="pr2_mechanism_model/SimpleTransmission" name="kinect_trans">
-    <actuator name="kinect_motor" />
-    <joint name="kinect_joint" />
-    <mechanicalReduction>1.0</mechanicalReduction>
-    <motorTorqueConstant>1.0</motorTorqueConstant>
-  </transmission-->
+  <gazebo reference="camera_link">
+    <sensor type="depth" name="openni_camera_camera">
+        <always_on>1</always_on>
+        <visualize>true</visualize>
+        <camera>
+            <horizontal_fov>1.047</horizontal_fov>
+            <image>
+                <width>640</width>
+                <height>480</height>
+                <format>R8G8B8</format>
+            </image>
+            <depth_camera>
+            </depth_camera>
+            <clip>
+                <near>0.1</near>
+                <far>100</far>
+            </clip>
+        </camera>
+        <plugin name="kinect_controller" filename="libgazebo_ros_openni_kinect.so">
+            <alwaysOn>true</alwaysOn>
+                <updateRate>10.0</updateRate>
+                <cameraName>cam3d</cameraName>
+                <frameName>camera_depth_optical_frame</frameName>
+            <imageTopicName>rgb/image_raw</imageTopicName>
+            <depthImageTopicName>depth/image_raw</depthImageTopicName>
+            <pointCloudTopicName>depth/points</pointCloudTopicName>
+            <cameraInfoTopicName>rgb/camera_info</cameraInfoTopicName>
+            <depthImageCameraInfoTopicName>depth/camera_info</depthImageCameraInfoTopicName>
+            <pointCloudCutoff>0.4</pointCloudCutoff>
+                <hackBaseline>0.07</hackBaseline>
+                <distortionK1>0.0</distortionK1>
+                <distortionK2>0.0</distortionK2>
+                <distortionK3>0.0</distortionK3>
+                <distortionT1>0.0</distortionT1>
+                <distortionT2>0.0</distortionT2>
+            <CxPrime>0.0</CxPrime>
+            <Cx>0.0</Cx>
+            <Cy>0.0</Cy>
+            <focalLength>0.0</focalLength>
+            </plugin>
+    </sensor>
+  </gazebo>
   <transmission name="kinect_trans">
     <type>transmission_interface/SimpleTransmission</type>
@@ -72,32 +58,34 @@
   </gazebo>
 </xacro:macro>
-<xacro:macro name="turtlebot_sim_imu_left">
-  <!--gazebo>
-    <controller:gazebo_ros_imu name="imu_controller" plugin="libgazebo_ros_imu.so">
+<!--xacro:macro name="turtlebot_sim_imu_left">
+ <gazebo>
+  <controller:gazebo_ros_imu name="imu_controller_left" plugin="libgazebo_ros_imu.so">
       <alwaysOn>true</alwaysOn>
       <updateRate>30</updateRate>
       <bodyName>imu_left_link</bodyName>
       <topicName>imu_left/data</topicName>
+      <serviceName>imu_left/service</serviceName>
       <gaussianNoise>${0.0017*0.0017}</gaussianNoise>
-      <xyzOffsets>0 0 0</xyzOffsets>
-      <rpyOffsets>0 0 0</rpyOffsets>
+      <xyzOffset>0 0 0</xyzOffset>
+      <rpyOffset>0 0 0</rpyOffset>
       <interface:position name="imu_left_position"/>
     </controller:gazebo_ros_imu>
-  </gazebo-->
+  </gazebo>
 </xacro:macro>
 <xacro:macro name="turtlebot_sim_imu_right">
-  <!--gazebo>
-    <controller:gazebo_ros_imu name="imu_controller" plugin="libgazebo_ros_imu.so">
+ <gazebo>
+  <controller:gazebo_ros_imu name="imu_controller_right" plugin="libgazebo_ros_imu.so">
       <alwaysOn>true</alwaysOn>
       <updateRate>30</updateRate>
       <bodyName>imu_right_link</bodyName>
       <topicName>imu_right/data</topicName>
+      <serviceName>imu_right/service</serviceName>
       <gaussianNoise>${0.0017*0.0017}</gaussianNoise>
-      <xyzOffsets>0 0 0</xyzOffsets>
-      <rpyOffsets>0 0 0</rpyOffsets>
+      <xyzOffset>0 0 0</xyzOffset>
+      <rpyOffset>0 0 0</rpyOffset>
       <interface:position name="imu_right_position"/>
     </controller:gazebo_ros_imu>
-  </gazebo-->
-</xacro:macro>
+  </gazebo>
+</xacro:macro-->
 <xacro:macro name="turtlebot_sim_laser">
   <!--gazebo reference="laser">
